File: datacenter-dram-tester.kicad_pcb (KiCad board)
At the start: 10 copper layers, 152.9 x 90 mm, 322 parts, among them IC1 TPS54561, IC3 TPD8S009DSMR, J1 0878311420, J10 61300311121, J3 DC_SOCKET, J4 WE_629105150521, J6 685119134923, J7 1140084168, J8 61300311121, Q2 BSS138APW, Q3 BSS138APW, Q4 BSS138APW, Q5 BSS138APW, Q6 BSS138APW, Q7 BSS138APW, Q8 BSS138APW, U10 LM3881MME_NOPB, U11 S27KL0641DABHI023, U12 TPS62823DLCT, U14 2199155-1, U15 XC7K160T-FFG676, U3 S25FL128SAGNFI000, U4 TPS65296, U5 TPS62823DLCT, U6 KSZ9031RNXCA, U7 FT4232HQ, U8 SRST, U9 TPS62823DLCT, Y1 ABM8G-25.000MHZ-18-D2Y-T, Y2 ABM8G-12.000MHZ-18-D2Y-T

Commit message: Update naming convention
Parts:
- 0V6, 1V1, 1V8, 3V3, 5V0, PUDC_B1, TP1, TP2, TP3, TP4, TP5, TP6, TP7, TP8, TP9, U8: footprint ddr4-datacenter-tester-footprints:Testpoint_smd_1mm -> datacenter-dram-tester-footprints:Testpoint_smd_1mm
- C1, C10, C100, C102, C109, C180, C182, C183, C2, C27, C28, C29, C31, C33, C37, C39, C4, C40, C41, C42, C45, C97, C98: footprint ddr4-datacenter-tester-footprints:0603-cap -> datacenter-dram-tester-footprints:0603-cap
- C101, C103, C104, C105, C119, C120, C121, C122, C123, C124, C125, C126, C127, C128, C129, C130, C131, C132, C133, C134, C135, C136, C137, C138, C139, C140, C141, C142, C147, C148, C149, C150, C151, C152, C172, C174, C175, C178, C184, C185, C186, C187, C188, C189, C190, C191, C192, C193, C194, C195, C196, C197, C198, C30, C35, C36, C38, C46, C5, C96, C99: footprint ddr4-datacenter-tester-footprints:0402-cap -> datacenter-dram-tester-footprints:0402-cap
- C116, C117, C118: footprint ddr4-datacenter-tester-footprints:1206-cap -> datacenter-dram-tester-footprints:1206-cap
- C20: footprint ddr4-datacenter-tester-footprints:KEMET_A -> datacenter-dram-tester-footprints:KEMET_A
- C26: footprint ddr4-datacenter-tester-footprints:KEMET_D -> datacenter-dram-tester-footprints:KEMET_D
- D1, D10, D5, D6, D7, D8, D9, PWR1: footprint ddr4-datacenter-tester-footprints:LED_0603 -> datacenter-dram-tester-footprints:LED_0603
- D11, D2: footprint ddr4-datacenter-tester-footprints:PDS760-13 -> datacenter-dram-tester-footprints:PDS760-13
- D3: footprint ddr4-datacenter-tester-footprints:SOT-3 -> datacenter-dram-tester-footprints:SOT-3
- D4: footprint ddr4-datacenter-tester-footprints:TPD6E05U06 -> datacenter-dram-tester-footprints:TPD6E05U06
- FB1, FB2, FB3, FB7, R38, R39, R41, R43, R44, R47, R48, R49, R85: footprint ddr4-datacenter-tester-footprints:0603-res -> datacenter-dram-tester-footprints:0603-res
- FB4, FB5, FB6: footprint ddr4-datacenter-tester-footprints:0603 -> datacenter-dram-tester-footprints:0603
- IC1: footprint ddr4-datacenter-tester-footprints:WSON-10_4x4 -> datacenter-dram-tester-footprints:WSON-10_4x4
- IC3: footprint ddr4-datacenter-tester-footprints:R-PDSO-N15 -> datacenter-dram-tester-footprints:R-PDSO-N15
- J1: footprint ddr4-datacenter-tester-footprints:PinHeader_2x7_P2mm_Drill1mm -> datacenter-dram-tester-footprints:PinHeader_2x7_P2mm_Drill1mm
- J10, J8, MODE2: footprint ddr4-datacenter-tester-footprints:PinHeader_1x3_P2.54_Drill1.1mm -> datacenter-dram-tester-footprints:PinHeader_1x3_P2.54_Drill1.1mm
- J3: footprint ddr4-datacenter-tester-footprints:DC_SOCKET -> datacenter-dram-tester-footprints:DC_SOCKET
- J4: footprint ddr4-datacenter-tester-footprints:USB_Micro_B_Female_629105150521 -> datacenter-dram-tester-footprints:USB_Micro_B_Female_629105150521
- J6: footprint ddr4-datacenter-tester-footprints:HDMI_A_Female_685119134923 -> datacenter-dram-tester-footprints:HDMI_A_Female_685119134923
- J7: footprint ddr4-datacenter-tester-footprints:MicroSD_1140084168 -> datacenter-dram-tester-footprints:MicroSD_1140084168
- J?1: footprint ddr4-datacenter-tester-footprints:7499111121A -> datacenter-dram-tester-footprints:7499111121A
- L1: footprint ddr4-datacenter-tester-footprints:IHLP2020BZER4R7M01 -> datacenter-dram-tester-footprints:IHLP2020BZER4R7M01
- L2: footprint ddr4-datacenter-tester-footprints:INDC3225X120N -> datacenter-dram-tester-footprints:INDC3225X120N
- L3, L4, L5: footprint ddr4-datacenter-tester-footprints:IHLP-1212AE -> datacenter-dram-tester-footprints:IHLP-1212AE
- L6: footprint ddr4-datacenter-tester-footprints:WE_7447798720 -> datacenter-dram-tester-footprints:WE_7447798720
- N1: footprint ddr4-datacenter-tester-footprints:oshw-logo -> datacenter-dram-tester-footprints:oshw-logo
- N2: footprint ddr4-datacenter-tester-footprints:antmicro-logo_scaled_20mm -> datacenter-dram-tester-footprints:antmicro-logo_scaled_20mm
- PROG_B1, USR_BTN1, USR_BTN2, USR_BTN3, USR_BTN4: footprint ddr4-datacenter-tester-footprints:Switch_Tactile_SMD_B3U-1000P -> datacenter-dram-tester-footprints:Switch_Tactile_SMD_B3U-1000P
- Q2, Q3, Q4, Q5, Q6, Q7, Q8: footprint ddr4-datacenter-tester-footprints:SC70-3 -> datacenter-dram-tester-footprints:SC70-3
- R1, R10, R11, R115, R116, R119, R12, R122, R126, R127, R128, R129, R13, R130, R131, R132, R133, R134, R135, R136, R137, R138, R139, R14, R140, R141, R142, R143, R144, R145, R146, R15, R16, R17, R18, R19, R2, R20, R21, R22, R23, R24, R25, R26, R27, R28, R29, R3, R30, R31, R32, R33, R34, R35, R36, R37, R4, R40, R42, R45, R5, R50, R51, R52, R53, R54, R55, R56, R57, R58, R59, R6, R60, R61, R62, R67, R68, R69, R7, R70, R71, R72, R73, R74, R75, R76, R77, R78, R79, R8, R80, R81, R82, R83, R84, R86, R87, R88, R89, R9, R90, R91, R92, R93, R94, R95, R96: footprint ddr4-datacenter-tester-footprints:0402-res -> datacenter-dram-tester-footprints:0402-res
- R100, R101, R102, R103, R104, R105, R106, R107, R108, R109, R110, R111, R112, R113, R114, R117, R118, R120, R121, R123, R124, R125, R147, R148, R149, R150, R151, R152, R153, R154, R155, R156, R157, R97, R98, R99: footprint ddr4-datacenter-tester-footprints:0201-res -> datacenter-dram-tester-footprints:0201-res
- R46: footprint ddr4-datacenter-tester-footprints:0402 -> datacenter-dram-tester-footprints:0402
- S1: footprint ddr4-datacenter-tester-footprints:Switch_Slide_11.6x4mm_EG1218 -> datacenter-dram-tester-footprints:Switch_Slide_11.6x4mm_EG1218
- U10: footprint ddr4-datacenter-tester-footprints:VSSOP8-Texas_Instruments-DGK0008A -> datacenter-dram-tester-footprints:VSSOP8-Texas_Instruments-DGK0008A
- U11: footprint ddr4-datacenter-tester-footprints:FBGA-24 -> datacenter-dram-tester-footprints:FBGA-24
- U12, U5, U9: footprint ddr4-datacenter-tester-footprints:QFN-8_2x1mm -> datacenter-dram-tester-footprints:QFN-8_2x1mm
- U14: footprint ddr4-datacenter-tester-footprints:2199155-1 -> datacenter-dram-tester-footprints:2199155-1
- U15: footprint ddr4-datacenter-tester-footprints:BGA676C100P26X26_2700X2700X254 -> datacenter-dram-tester-footprints:BGA676C100P26X26_2700X2700X254
- U3: footprint ddr4-datacenter-tester-footprints:S25FL128SAGNFI000 -> datacenter-dram-tester-footprints:S25FL128SAGNFI000
- U4: footprint ddr4-datacenter-tester-footprints:VQFN-HR -> datacenter-dram-tester-footprints:VQFN-HR
- U6: footprint ddr4-datacenter-tester-footprints:QFN-48-Microchip-QFN77-48LD-PL-2 -> datacenter-dram-tester-footprints:QFN-48-Microchip-QFN77-48LD-PL-2
- U7: footprint ddr4-datacenter-tester-footprints:FT4232HQ -> datacenter-dram-tester-footprints:FT4232HQ
- Y1, Y2: footprint ddr4-datacenter-tester-footprints:KX-7 -> datacenter-dram-tester-footprints:KX-7
