File: data-center-dram-tester.kicad_pcb (KiCad board)
At the start: 10 copper layers, 152.9 x 90 mm, 430 parts, among them IC1 TPS54561, IC3 TPD8S009DSMR, J1 0878311420, J3 DC_SOCKET, J4 WE_629105150521, J6 685119134923, J7 1140084168, J8 61300311121, Q2 BSS138APW, Q3 BSS138APW, Q4 BSS138APW, Q5 BSS138APW, Q6 BSS138APW, Q7 BSS138APW, Q8 BSS138APW, U1 ASFLMB-100.000MHZ-XY-T, U10 LM3881MME_NOPB, U11 S27KL0641DABHI023, U12 TPS62823DLCT, U14 2199155-1, U15 XC7K160T-FFG676, U2 TPS65295RJET, U3 S25FL128SAGNFI000, U4 TPS62823DLCT, U5 TPS62823DLCT, U6 KSZ9031RNXCA, U7 FT4232HQ, U8 SRST, U9 TPS62823DLCT, Y1 ABM8G-25.000MHZ-18-D2Y-T, Y2 ABM8G-12.000MHZ-18-D2Y-T

Commit message: Add debug USB layout
Routing:
- net AUX_JTAG_TCK: track 5.31 -> 28.9 mm
- net AUX_JTAG_TDI: track 6.01 -> 29.2 mm
- net AUX_JTAG_TDO: track 3.12 -> 25.5 mm
- net AUX_JTAG_TMS: track 5.98 -> 27.3 mm
- net UART0_RX: track 15.1 -> 36.3 mm
- net UART0_TX: track 15.1 -> 35.3 mm
- net UART1_RX: track 23.5 -> 43.7 mm
- net UART1_TX: track 24.1 -> 44.1 mm
- net LED_SPD: track 28.2 -> 44.7 mm
