File: supply.kicad_sch (KiCad schematic)
At the start: 192 parts, among them IC1 TPS54561, J3 DC_SOCKET, J8 61300311121, Q11 BSS138APW, Q12 BSS138APW, U10 LM3881MME_NOPB, U12 AP62301WU-7, U17 74LVC2G07GV, U18 MAX812REUS+T, U19 PAC1954T-E/4MX, U2 TPS65295RJET, U20 PAC1954T-E/4MX, U21 SN74AHCT1G125DBVR, U22 SN74AHCT1G125DBVR, U23 SN74AHCT1G125DBVR, U24 74LVC2G07GV, U25 NCP718ASN500T1G, U26 MAX16150AUT+T, U27 SN74LVC1G240DCKR, U4 AP62301WU-7, U5 AP62301WU-7, U9 AP62301WU-7

Commit message: Optimize BOM, add all bank 115 and 116 REFCLK's to FMC connector
Parts:
- IC1: value TPS54561 -> TPS54561QDPRRQ1; footprint data-center-dram-tester-footprints:WSON-10_4x4 -> antmicro-footprints:WSON-10_4x4; symbol data-center-dram-tester:TPS54561 -> antmicroPMICVoltageRegulatorsLinear:TPS54561QDPRRQ1; MPN TPS54561-Q1 -> TPS54561QDPRRQ1
- R198, R200, R201, R202, R203, R204: MPN ERJMP2KF10MU -> RL1206FR-7W0R01L; Manufacturer PANASONIC -> Yageo
Other:
- note removed: "TODO: Find Replacement for 0R01"
- note removed: "TODO: Replace TPS54561 with TPS54561QDPRRQ1"
Changed lines of the file:
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@@
     (effects (font (size 1 1)) (justify left bottom))
   )
-  (text "TODO: Replace TPS54561 with TPS54561QDPRRQ1" (at 424.18 120.65 0)
-    (effects (font (size 1.27 1.27)) (justify left bottom))
-  )
   (text "VCC5V0 4.5V to 5.5V" (at 13.97 23.495 0)
     (effects (font (size 1.27 1.27)) (justify left bottom))
@@
     (effects (font (size 1 1)) (justify left bottom))
   )
-  (text "TODO: Find Replacement for 0R01 " (at 424.18 118.11 0)
-    (effects (font (size 1.27 1.27)) (justify left bottom))
-  )
   (text "Power Monitors" (at 320.04 114.935 0)
     (effects (font (size 2.0066 2.0066) (thickness 0.4013) bold) (justify left bottom))
@@
     (pin "1")
   )
-  (symbol (lib_id "data-center-dram-tester:TPS54561") (at 88.9 147.32 0) (unit 1)
+  (symbol (lib_id "antmicroPMICVoltageRegulatorsLinear:TPS54561QDPRRQ1") (at 88.9 147.32 0) (unit 1)
     (in_bom yes) (on_board yes)
     (property "Reference" "IC1" (id 0) (at 80.645 133.35 0)
       (effects (font (size 1.524 1.524)))
     )
-    (property "Value" "TPS54561" (id 1) (at 84.455 163.83 0)
-      (effects (font (size 1.524 1.524)))
+    (property "Value" "TPS54561QDPRRQ1" (id 1) (at 78.74 165.1 0)
+      (effects (font (size 1.524 1.524)) (justify left bottom))
     )
-    (property "Footprint" "data-center-dram-tester-footprints:WSON-10_4x4" (id 2) (at 88.9 147.32 0)
+    (property "Footprint" "antmicro-footprints:WSON-10_4x4" (id 2) (at 88.9 147.32 0)
       (effects (font (size 1.524 1.524)) hide)
     )
@@
       (effects (font (size 1.27 1.27)) hide)
     )
-    (property "MPN" "TPS54561-Q1" (id 5) (at 88.9 147.32 0)
+    (property "MPN" "TPS54561QDPRRQ1" (id 5) (at 88.9 147.32 0)
       (effects (font (size 1.27 1.27)) hide)
     )
@@
     (pin "2")
   )
-  (symbol (lib_id "antmicroResistorsmisc:R_0R01_1206") (at 383.54 187.325 0) (unit 1)
+  (symbol (lib_name "R_0R01_1206_3") (lib_id "antmicroResistorsmisc:R_0R01_1206") (at 383.54 187.325 0) (unit 1)
     (in_bom yes) (on_board yes)
     (property "Reference" "R202" (id 0) (at 377.825 185.42 0)
@@
       (effects (font (size 1.27 1.27)) hide)
     )
-    (property "Manufacturer" "PANASONIC" (id 4) (at 388.62 177.165 0)
+    (property "Manufacturer" "Yageo" (id 4) (at 388.62 177.165 0)
       (effects (font (size 1.524 1.524)) (justify left) hide)
     )
-    (property "MPN" "ERJMP2KF10MU" (id 5) (at 388.62 179.705 0)
+    (property "MPN" "RL1206FR-7W0R01L" (id 5) (at 388.62 179.705 0)
       (effects (font (size 1.524 1.524)) (justify left) hide)
     )
@@
     (pin "2")
   )
-  (symbol (lib_id "antmicroResistorsmisc:R_0R01_1206") (at 383.54 206.375 0) (unit 1)
+  (symbol (lib_name "R_0R01_1206_5") (lib_id "antmicroResistorsmisc:R_0R01_1206") (at 383.54 206.375 0) (unit 1)
     (in_bom yes) (on_board yes)
     (property "Reference" "R204" (id 0) (at 377.825 204.47 0)
@@
       (effects (font (size 1.27 1.27)) hide)
     )
-    (property "Manufacturer" "PANASONIC" (id 4) (at 388.62 196.215 0)
+    (property "Manufacturer" "Yageo" (id 4) (at 388.62 196.215 0)
       (effects (font (size 1.524 1.524)) (justify left) hide)
     )
-    (property "MPN" "ERJMP2KF10MU" (id 5) (at 388.62 198.755 0)
+    (property "MPN" "RL1206FR-7W0R01L" (id 5) (at 388.62 198.755 0)
       (effects (font (size 1.524 1.524)) (justify left) hide)
     )
@@
     (pin "1")
   )
-  (symbol (lib_id "antmicroResistorsmisc:R_0R01_1206") (at 383.54 127.635 0) (unit 1)
+  (symbol (lib_name "R_0R01_1206_1") (lib_id "antmicroResistorsmisc:R_0R01_1206") (at 383.54 127.635 0) (unit 1)
     (in_bom yes) (on_board yes)
     (property "Reference" "R198" (id 0) (at 377.825 125.73 0)
@@
       (effects (font (size 1.27 1.27)) hide)
     )
-    (property "Manufacturer" "PANASONIC" (id 4) (at 388.62 117.475 0)
+    (property "Manufacturer" "Yageo" (id 4) (at 388.62 117.475 0)
       (effects (font (size 1.524 1.524)) (justify left) hide)
     )
-    (property "MPN" "ERJMP2KF10MU" (id 5) (at 388.62 120.015 0)
+    (property "MPN" "RL1206FR-7W0R01L" (id 5) (at 388.62 120.015 0)
       (effects (font (size 1.524 1.524)) (justify left) hide)
     )
@@
     (pin "1")
   )
-  (symbol (lib_id "antmicroResistorsmisc:R_0R01_1206") (at 383.54 146.685 0) (unit 1)
+  (symbol (lib_name "R_0R01_1206_2") (lib_id "antmicroResistorsmisc:R_0R01_1206") (at 383.54 146.685 0) (unit 1)
     (in_bom yes) (on_board yes)
     (property "Reference" "R200" (id 0) (at 377.825 144.78 0)
@@
       (effects (font (size 1.27 1.27)) hide)
     )
-    (property "Manufacturer" "PANASONIC" (id 4) (at 388.62 136.525 0)
+    (property "Manufacturer" "Yageo" (id 4) (at 388.62 136.525 0)
       (effects (font (size 1.524 1.524)) (justify left) hide)
     )
-    (property "MPN" "ERJMP2KF10MU" (id 5) (at 388.62 139.065 0)
+    (property "MPN" "RL1206FR-7W0R01L" (id 5) (at 388.62 139.065 0)
       (effects (font (size 1.524 1.524)) (justify left) hide)
     )
@@
     (pin "2")
   )
-  (symbol (lib_id "antmicroResistorsmisc:R_0R01_1206") (at 383.54 196.85 0) (unit 1)
+  (symbol (lib_name "R_0R01_1206_4") (lib_id "antmicroResistorsmisc:R_0R01_1206") (at 383.54 196.85 0) (unit 1)
     (in_bom yes) (on_board yes)
     (property "Reference" "R203" (id 0) (at 377.825 194.945 0)
@@
       (effects (font (size 1.27 1.27)) hide)
     )
-    (property "Manufacturer" "PANASONIC" (id 4) (at 388.62 186.69 0)
+    (property "Manufacturer" "Yageo" (id 4) (at 388.62 186.69 0)
       (effects (font (size 1.524 1.524)) (justify left) hide)
     )
-    (property "MPN" "ERJMP2KF10MU" (id 5) (at 388.62 189.23 0)
+    (property "MPN" "RL1206FR-7W0R01L" (id 5) (at 388.62 189.23 0)
       (effects (font (size 1.524 1.524)) (justify left) hide)
     )
@@
       (effects (font (size 1.27 1.27)) hide)
     )
-    (property "Manufacturer" "PANASONIC" (id 4) (at 388.62 167.64 0)
+    (property "Manufacturer" "Yageo" (id 4) (at 388.62 167.64 0)
       (effects (font (size 1.524 1.524)) (justify left) hide)
     )
-    (property "MPN" "ERJMP2KF10MU" (id 5) (at 388.62 170.18 0)
+    (property "MPN" "RL1206FR-7W0R01L" (id 5) (at 388.62 170.18 0)
       (effects (font (size 1.524 1.524)) (justify left) hide)
     )
