File: DDR4.kicad_sch (KiCad schematic)
At the start: 39 parts, among them U14 2199155-1

Commit message: Loclib of the project
Parts:
- C153, C154, C160, C161, C162, C163, C164, C165, C166, C167, C168, C169, C170, C171, C173, C176, C177, C179, C181, C199, C200, C201, C202, C203, C204, C205, C208, C209, C210, C211, C212, C213, C214: footprint antmicro-footprints:0402-cap -> data-center-dram-tester-footprints:0402-cap; symbol antmicroCapacitors0402:C_100n_0402 -> data-center-dram-tester:C_100n_0402
- R157, R158, R185: footprint antmicro-footprints:0402-res -> data-center-dram-tester-footprints:0402-res; symbol antmicroResistors0402:R_0R_0402 -> data-center-dram-tester:R_0R_0402
- R186: footprint antmicro-footprints:0402-res -> data-center-dram-tester-footprints:0402-res; symbol antmicroResistors0402:R_100k_0402 -> data-center-dram-tester:R_100k_0402
