File: fpga-banks-12-15.kicad_sch (KiCad schematic)
At the start: 1 part, among them U15 XC7K160T-FFG676

Commit message: Loclib of the project
Parts:
- U15: footprint antmicro-footprints:xc7k160tfbg676 -> data-center-dram-tester-footprints:xc7k160tfbg676
