File: hyperram.kicad_sch (KiCad schematic)
At the start: 7 parts, among them U11 S27KL0641DABHI023

Commit message: Loclib of the project
Parts:
- C103, C104, C105: footprint antmicro-footprints:0402-cap -> data-center-dram-tester-footprints:0402-cap; symbol antmicroCapacitors0402:C_100n_0402 -> data-center-dram-tester:C_100n_0402
